File: arisu.kicad_pcb (KiCad board)
At the start: 2 copper layers, 339.1 x 118.7 mm, 176 parts, among them J1 USB_B_Micro, SW1 SW_Push, SW10 SW_Push, SW11 SW_Push, SW12 SW_Push, SW13 SW_Push, SW14 SW_Push, SW15 SW_Push, SW16 SW_Push, SW17 SW_Push, SW18 SW_Push, SW19 SW_Push, SW2 SW_Push, SW20 SW_Push, SW21 SW_Push, SW22 SW_Push, SW23 SW_Push, SW24 SW_Push, SW25 SW_Push, SW26 SW_Push, SW27 SW_Push, SW28 SW_Push, SW29 SW_Push, SW3 SW_Push, SW30 SW_Push, SW31 SW_Push, SW32 SW_Push, SW33 SW_Push, SW34 SW_Push, SW35 SW_Push, SW36 SW_Push, SW37 SW_Push, SW38 SW_Push, SW39 SW_Push, SW4 SW_Push, SW40 SW_Push, SW41 SW_Push, SW42 SW_Push, SW43 SW_Push, SW44 SW_Push, SW45 SW_Push, SW46 SW_Push, SW47 SW_Push, SW48 SW_Push, SW49 SW_Push, SW5 SW_Push, SW50 SW_Push, SW51 SW_Push, SW52 SW_Push, SW53 SW_Push, SW54 SW_Push, SW55 SW_Push, SW56 SW_Push, SW57 SW_Push, SW58 SW_Push, SW59 SW_Push, SW6 SW_Push, SW60 SW_Push, SW61 SW_Push, SW62 SW_Push, SW63 SW_Push, SW64 SW_Push, SW65 SW_Push, SW66 SW_Push, SW67 SW_Push, SW7 SW_Push, SW8 SW_Push, SW9 SW_Push, U1 USBLC6-2SC6, U2 ATmega32U4-AU, Y1 Crystal_GND24

Commit message: WIP Neito
Parts:
- removed the G*** at (287.0, 114.9)
- removed the G*** at (287.0, 117.3)
- removed J1: USB_B_Micro, Connectors_USB:USB_Micro-B_Molex-105017-0001
- added D68: D, Diode_SMD:D_SOD-123, B.Cu at (55.5, 101.3)
- added ENC0: Rotary_Encoder_Switch, Keebio-Parts:RotaryEncoder_EC11, F.Cu at (350.8, 34.0)
- added G***: LOGO, pohjola:Neito(nate), F.Cu at (286.8, 116.0)
- added G***: LOGO, pohjola:pohjola_site_text, B.Cu at (69.9, 115.5)
- added G***: LOGO, pohjola:pohjola_text, B.Cu at (287.1, 117.1)
- added R_CC1: 5.1k, keyboard_parts:R_2012, B.Cu at (186.5, 27.6)
- added R_CC2: 5.1k, keyboard_parts:R_2012, B.Cu at (190.1, 27.6)
- added SW68: SW_Push, MX_Switch:MX_1.00u_PCB, F.Cu at (58.8, 95.9)
- added USB_C1: USB_C_Receptacle_HRO_TYPE-C-31-M-12, USB_Type-C:USB_C_Receptacle_HRO_TYPE-C-31-M-12-HandSoldering, F.Cu at (175.1, 22.9)
- SW4: footprint Fate_Parts:SW_Cherry_MX_2.25u_PCB -> MX_Switch:SW_Cherry_MX_1.25u_PCB
- SW57: footprint Fate_Parts:SW_Cherry_MX_2.25u_PCB_ReversedStabilizers -> MX_Switch:SW_Cherry_MX_1.00u_PCB
- SW60: footprint Fate_Parts:SW_Cherry_MX_1.50u_PCB -> MX_Switch:SW_Cherry_MX_2.00u_PCB
- moved SW60 30.5 mm to (338.3, 48.2), turned to 270 degrees
- moved D57 11.9 mm to (304.1, 80.6)
- moved D4 9.52 mm to (34.1, 99.6)
- moved D60 6.72 mm to (325.0, 64.3), turned to 0 degrees
- moved D55 4.27 mm to (285.7, 42.5)
- moved D56 4.27 mm to (299.4, 61.5)
- moved SW59 4.27 mm to (298.4, 29.2)
- moved D51 4.27 mm to (266.6, 41.0)
- moved D52 4.27 mm to (280.3, 61.5)
- moved D59 4.27 mm to (304.7, 42.5)
- moved D64 4.27 mm to (347.6, 37.7)
- moved D65 4.27 mm to (351.8, 56.8)
- moved D66 4.27 mm to (356.0, 75.8)
- moved H7 4.27 mm to (345.4, 43.5)
- moved SW51 4.27 mm to (260.3, 27.7)
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- renumbered PF6 to J10, PF7 to J11, VCC to J12, D+ to J13, D- to J14, GND to J15, MISO to J2, VCC to J3, SCK to J4, MOSI to J5, RES to J6, GND to J7, PF4 to J8, PF5 to J9
Routing:
- net /PF5: track 40.2 -> 231.5 mm, vias 1 -> 3
- net /PF4: track 38.1 -> 223.0 mm, vias 1 -> 3
- net GND: track 71.6 -> 230.6 mm
- net Net-(R_CC2-Pad1): track 0.00 -> 24.7 mm, vias 0 -> 1
- net Net-(J14-Pad1): track 45.1 -> 66.7 mm
- net /col1: track 166.8 -> 185.9 mm
- net /row4: track 433.8 -> 451.6 mm
- net /row3: track 432.5 -> 446.4 mm
- net Net-(R_CC1-Pad2): track 0.00 -> 13.4 mm, vias 0 -> 1
- net /col13: track 269.0 -> 276.6 mm
- net Net-(D68-Pad2): track 0.00 -> 6.56 mm
- net Net-(D63-Pad2): track 4.91 -> 10.9 mm
- net Net-(J13-Pad1): track 47.8 -> 53.7 mm, vias 0 -> 1
- net VCC: track 205.4 -> 210.9 mm
- net /row1: track 384.1 -> 388.6 mm
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Other:
- board size 339.1 x 118.7 mm -> 343.4 x 118.7 mm
- board text removed: "Fate Design Rev 1.1"
